File: thinkeys.kicad_pcb (KiCad board)
At the start: 2 copper layers, 330.6 x 266.1 mm, 403 parts, among them J1 Pointing stick, J2 Pointing stick, J3 PWRSWITCH, J4 Conn_01x03_Male, J5 Conn_01x01_Female, J6 Conn_01x01_Female, SW1 SW_Push, SW10 SW_Push, SW11 SW_Push, SW12 SW_Push, SW13 SW_Push, SW14 SW_Push, SW15 SW_Push, SW16 SW_Push, SW17 SW_Push, SW18 SW_Push, SW19 SW_Push, SW2 SW_Push, SW20 SW_Push, SW21 SW_Push, SW22 SW_Push, SW23 SW_Push, SW24 SW_Push, SW25 SW_Push, SW26 SW_Push, SW27 SW_Push, SW28 SW_Push, SW29 SW_Push, SW3 SW_Push, SW30 SW_Push, SW31 SW_Push, SW32 SW_Push, SW33 SW_Push, SW34 SW_Push, SW35 SW_Push, SW36 SW_Push, SW37 SW_Push, SW38 SW_Push, SW39 SW_Push, SW4 SW_Push, SW40 SW_Push, SW41 SW_Push, SW42 SW_Push, SW43 SW_Push, SW44 SW_Push, SW45 SW_Push, SW46 SW_Push, SW47 SW_Push, SW48 SW_Push, SW49 SW_Push, SW5 SW_Push, SW50 SW_Push, SW51 SW_Push, SW54 SW_Push, SW55 SW_Push, SW56 SW_Push, SW57 SW_Push, SW58 SW_Push, SW59 SW_Push, SW6 SW_Push, SW60 SW_Push, SW61 SW_Push, SW62 SW_Push, SW63 SW_Push, SW64 SW_Push, SW65 SW_Push, SW66 SW_Push, SW69 SW_Push, SW7 SW_Push, SW70 SW_Push, SW71 SW_Push, SW72 SW_Push, SW73 SW_Push, SW74 SW_Push, SW75 SW_Push, SW76 SW_Push, SW77 SW_Push, SW78 SW_Push, SW79 SW_Push, SW8 SW_Push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

Commit message: R11: 4.7 kΩ to 100 kΩ
Parts:
- R11: value 4.7k -> 100k
Connections:
- U1 pad 24: Net-(U1-Pad24) -> (no net)
- U1 pad 25: Net-(U1-Pad25) -> (no net)
- U1 pad 27: Net-(U1-Pad27) -> (no net)
- U1 pad 28: Net-(U1-Pad28) -> (no net)
- U1 pad 29: Net-(U1-Pad29) -> (no net)
- U2 pad 24: Net-(U2-Pad24) -> (no net)
- U2 pad 25: Net-(U2-Pad25) -> (no net)
- U2 pad 27: Net-(U2-Pad27) -> (no net)
- U2 pad 28: Net-(U2-Pad28) -> (no net)
- U2 pad 29: Net-(U2-Pad29) -> (no net)
- USB1 pad 10: Net-(USB1-Pad10) -> (no net)
- USB1 pad 3: Net-(USB1-Pad3) -> (no net)
- USB1 pad 4: Net-(USB1-Pad4) -> (no net)
- USB1 pad 9: Net-(USB1-Pad9) -> (no net)
- USB2 pad 10: Net-(USB2-Pad10) -> (no net)
- USB2 pad 3: Net-(USB2-Pad3) -> (no net)
- USB2 pad 4: Net-(USB2-Pad4) -> (no net)
- USB2 pad 9: Net-(USB2-Pad9) -> (no net)

Commit message: pcb: use updated pointing stick footprints
Parts:
- moved REF** 0.35 mm to (178.5, 177.3)
- moved J2 0.35 mm to (178.5, 29.3)
- moved J1 0.35 mm to (112.3, 38.1)
- moved REF** 0.35 mm to (112.3, 157.1)
Other:
- outline, holes or cut-outs redrawn

Commit message: pcb: switch to cardioid style castellated landing
Parts:
- TP1, TP13, TP14, TP15, TP16, TP17, TP18, TP2, TP25, TP26, TP27, TP28, TP29, TP3, TP30, TP31, TP39, TP4, TP40, TP41, TP42, TP43, TP44, TP45, TP46, TP5, TP6: footprint libmodulo:SMDPad_4.0x2.0mm -> libmodulo:SMDPad_2.0mm
Routing:
- net /right/r0: track 173.1 -> 171.8 mm
- net /right/c7: track 134.9 -> 133.6 mm
- net /right/c6: track 127.1 -> 125.8 mm
- net /right/c3: track 103.2 -> 101.9 mm
- net /left/r0: track 135.9 -> 134.6 mm
- net /left/c3: track 90.5 -> 89.2 mm
- net /left/c1: track 105.1 -> 103.9 mm
- net /left/c0: track 112.9 -> 111.7 mm
- net /left/r5: track 46.7 -> 45.4 mm
- net /left/r3: track 41.6 -> 40.4 mm
- net /left/r2: track 39.1 -> 37.8 mm
- net /left/c6: track 64.3 -> 63.0 mm
- net /right/r5: track 66.1 -> 64.8 mm
- net /right/r4: track 63.5 -> 62.3 mm
- net /right/r3: track 61.0 -> 59.7 mm
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
Commit message: pcb: tab screw M1 to M1.6
Parts:
- ? (x3): value (none) -> Val**; footprint (none) -> libmodulo:JIS_M1.6
- REF** (x3): footprint libmodulo:m1 -> libmodulo:JIS_M1.6

Commit message: pcb: kicad 6
Other:
- outline, holes or cut-outs redrawn
- net class Default removed
- net class power removed
